Commit message: [Mini Quadrotor][Experiment]Preparations
Add the camera into urdf file. Delete the camera in gazebo.

File: robots/mini_quadrotor/urdf/robot.gazebo.xacro (robot description, xacro)
@@ -54,27 +54,4 @@
   <!-- </gazebo> -->
   <!-- sensors -->
-  <!-- 1. stereo camera: depth, color based on left camera -->
-  <xacro:extra_module name = "downward_camera_frame" parent = "main_body">
-    <origin xyz="0.0 0.00 -0.05" rpy="0 ${pi/2} 0"/>
-    <inertial>
-      <mass value = "0.00001" />
-      <origin xyz="0 0 0" rpy="0 0 0"/>
-      <inertia
-          ixx="0.000001" ixy="0.0" ixz="0.0"
-          iyy="0.000001" iyz="0.0"
-          izz="0.000002"/>
-    </inertial>
-  </xacro:extra_module>
-  <xacro:extra_module name = "downward_camera_optical_frame" parent = "downward_camera_frame">
-    <origin xyz="0 0 0" rpy="${-pi / 2} 0 ${-pi / 2}"/>
-    <inertial>
-      <mass value = "0.00001" />
-      <origin xyz="0 0 0" rpy="0 0 0"/>
-      <inertia
-          ixx="0.000001" ixy="0.0" ixz="0.0"
-          iyy="0.000001" iyz="0.0"
-          izz="0.000002"/>
-    </inertial>
-  </xacro:extra_module>
   <!-- gazebo plugin -->
   <gazebo reference="downward_camera_frame">

File: robots/mini_quadrotor/urdf/robot.urdf.xacro (robot description, xacro)
@@ -183,4 +183,27 @@
     </inertial>
   </xacro:extra_module>
+  <!-- downward camera: depth, color based on left camera -->
+  <xacro:extra_module name = "downward_camera_frame" parent = "main_body">
+    <origin xyz="0.0 0.00 -0.05" rpy="0 ${pi/2} 0"/>
+    <inertial>
+      <mass value = "0.00001" />
+      <origin xyz="0 0 0" rpy="0 0 0"/>
+      <inertia
+          ixx="0.000001" ixy="0.0" ixz="0.0"
+          iyy="0.000001" iyz="0.0"
+          izz="0.000002"/>
+    </inertial>
+  </xacro:extra_module>
+  <xacro:extra_module name = "downward_camera_optical_frame" parent = "downward_camera_frame">
+    <origin xyz="0 0 0" rpy="${-pi / 2} 0 ${-pi / 2}"/>
+    <inertial>
+      <mass value = "0.00001" />
+      <origin xyz="0 0 0" rpy="0 0 0"/>
+      <inertia
+          ixx="0.000001" ixy="0.0" ixz="0.0"
+          iyy="0.000001" iyz="0.0"
+          izz="0.000002"/>
+    </inertial>
+  </xacro:extra_module>
   <!-- propellers -->
   <xacro:propeller_module id = "1" x = "${-rotor_x}" y = "${-rotor_y}" z = "${rotor_z}" direction = "-1" />
