Commit message: [Mini Quadrotor][Apriltag] Change the bundle tags in gazebo
1. Change the Tag zero to a bundle of tags(1-2-0-3-4). But the posture of these tags is incorrect.
2.Remap the name of topics to make it same with the camera's topic in simulation.
3. Change the frame's name of tags. Because now I'm using a bundle of tags.
4. Change the position of camera of the model.

File: robots/mini_quadrotor/urdf/robot.urdf.xacro (robot description, xacro)
@@ -185,5 +185,5 @@
   <!-- downward camera: depth, color based on left camera -->
   <xacro:extra_module name = "downward_camera_frame" parent = "main_body">
-    <origin xyz="0.0 0.00 -0.05" rpy="0 ${pi/2} 0"/>
+    <origin xyz="0.077 -0.01 -0.012" rpy="0 ${pi/2} 0"/>
     <inertial>
       <mass value = "0.00001" />

Commit message: [Mini_Quadrotor][Code]Install the camera so change some files
1.Set the size of real apriltag
2.Change the parameter of camera
3.Change the position of coordinate of camera

File: robots/mini_quadrotor/urdf/robot.urdf.xacro (robot description, xacro)
@@ -185,5 +185,5 @@
   <!-- downward camera: depth, color based on left camera -->
   <xacro:extra_module name = "downward_camera_frame" parent = "main_body">
-    <origin xyz="0.077 -0.01 -0.012" rpy="0 ${pi/2} 0"/>
+    <origin xyz="0.0925 0.00 -0.017" rpy="0 ${pi/2} 0"/>
     <inertial>
       <mass value = "0.00001" />

Commit message: [MIni_Quadrotor][config] Add the mess of camera case in the urdf file.
And change the flag of Apriltag

File: robots/mini_quadrotor/urdf/robot.urdf.xacro (robot description, xacro)
@@ -187,5 +187,5 @@
     <origin xyz="0.0925 0.00 -0.017" rpy="0 ${pi/2} 0"/>
     <inertial>
-      <mass value = "0.00001" />
+      <mass value = "0.080" />
       <origin xyz="0 0 0" rpy="0 0 0"/>
       <inertia

Commit message: [Mini_Quadrotor][code] Move to a new repository

File: robots/mini_quadrotor/urdf/robot.urdf.xacro (robot description, xacro)
@@ -187,10 +187,10 @@
     <origin xyz="0.0925 0.00 -0.017" rpy="0 ${pi/2} 0"/>
     <inertial>
-      <mass value = "0.080" />
+      <mass value = "0.00001" />
       <origin xyz="0 0 0" rpy="0 0 0"/>
       <inertia
           ixx="0.000001" ixy="0.0" ixz="0.0"
           iyy="0.000001" iyz="0.0"
-          izz="0.000002"/>
+          izz="0.000002"/>-->
     </inertial>
   </xacro:extra_module>
@@ -198,6 +198,6 @@
     <origin xyz="0 0 0" rpy="${-pi / 2} 0 ${-pi / 2}"/>
     <inertial>
-      <mass value = "0.00001" />
-      <origin xyz="0 0 0" rpy="0 0 0"/>
+     <mass value = "0.00001" />
+     <origin xyz="0 0 0" rpy="0 0 0"/>
       <inertia
           ixx="0.000001" ixy="0.0" ixz="0.0"

Commit message: [Mini_Quadrotor][launch] Add a apriltag frame

File: robots/mini_quadrotor/urdf/robot.urdf.xacro (robot description, xacro)
@@ -184,6 +184,28 @@
   </xacro:extra_module>
   <!-- downward camera: depth, color based on left camera -->
-  <xacro:extra_module name = "downward_camera_frame" parent = "main_body">
-    <origin xyz="0.0925 0.00 -0.017" rpy="0 ${pi/2} 0"/>
+  <!-- <xacro:extra_module name = "downward_camera_frame" parent = "main_body"> -->
+  <!--   <origin xyz="0.0925 0.00 -0.017" rpy="0 ${pi/2} 0"/> -->
+  <!--   <inertial> -->
+  <!--     <mass value = "0.00001" /> -->
+  <!--     <origin xyz="0 0 0" rpy="0 0 0"/> -->
+  <!--     <inertia -->
+  <!--         ixx="0.000001" ixy="0.0" ixz="0.0" -->
+  <!--         iyy="0.000001" iyz="0.0" -->
+  <!--         izz="0.000002"/>-\-> -->
+  <!--   </inertial> -->
+  <!-- </xacro:extra_module> -->
+  <!-- <xacro:extra_module name = "downward_camera_optical_frame" parent = "downward_camera_frame"> -->
+  <!--   <origin xyz="0 0 0" rpy="${-pi / 2} 0 ${-pi / 2}"/> -->
+  <!--   <inertial> -->
+  <!--    <mass value = "0.00001" /> -->
+  <!--    <origin xyz="0 0 0" rpy="0 0 0"/> -->
+  <!--     <inertia -->
+  <!--         ixx="0.000001" ixy="0.0" ixz="0.0" -->
+  <!--         iyy="0.000001" iyz="0.0" -->
+  <!--         izz="0.000002"/> -->
+  <!--   </inertial> -->
+  <!-- </xacro:extra_module> -->
+  <xacro:extra_module name = "Apriltag_frame" parent = "main_body">
+    <origin xyz=" 0.173 0.00 -0.008" rpy="0 ${pi} 0"/>
     <inertial>
       <mass value = "0.00001" />
@@ -193,15 +215,4 @@
           iyy="0.000001" iyz="0.0"
           izz="0.000002"/>-->
-    </inertial>
-  </xacro:extra_module>
-  <xacro:extra_module name = "downward_camera_optical_frame" parent = "downward_camera_frame">
-    <origin xyz="0 0 0" rpy="${-pi / 2} 0 ${-pi / 2}"/>
-    <inertial>
-     <mass value = "0.00001" />
-     <origin xyz="0 0 0" rpy="0 0 0"/>
-      <inertia
-          ixx="0.000001" ixy="0.0" ixz="0.0"
-          iyy="0.000001" iyz="0.0"
-          izz="0.000002"/>
     </inertial>
   </xacro:extra_module>

Commit message: [Qilin][simulation] Add the apriltag
There is a problem. I can see apriltag in rviz but cannot see in gazebo.

File: robots/mini_quadrotor/urdf/robot.urdf.xacro (robot description, xacro)
@@ -206,15 +206,44 @@
   <!--   </inertial> -->
   <!-- </xacro:extra_module> -->
-  <xacro:extra_module name = "Apriltag_frame" parent = "main_body">
-    <origin xyz=" 0.173 0.00 -0.008" rpy="0 ${pi} 0"/>
-    <inertial>
-      <mass value = "0.00001" />
-      <origin xyz="0 0 0" rpy="0 0 0"/>
-      <inertia
-          ixx="0.000001" ixy="0.0" ixz="0.0"
-          iyy="0.000001" iyz="0.0"
-          izz="0.000002"/>-->
-    </inertial>
-  </xacro:extra_module>
+  <!-- New link for the AprilTag -->
+  <link name="apriltag_link">
+    <visual>
+      <origin xyz="0 0 0" rpy="${-pi} 0 0"/>
+      <geometry>
+        <box size="0.032 0.032 0.001"/>
+      </geometry>
+      <material name="apriltag_material">
+        <texture filename="package://aerial_robot_simulation/gazebo_model/models/Apriltag36_11_00000/materials/textures/tag36_11_00000.png"/>
+      </material>
+    </visual>
+    <collision>
+      <origin xyz="0 0 0" rpy="0 0 0"/>
+      <geometry>
+        <box size="0.032 0.032 0.001"/>
+      </geometry>
+    </collision>
+    <inertial>
+      <mass value="0.01"/>
+      <origin xyz="0 0 0"/>
+      <inertia ixx="0.0001" ixy="0.0" ixz="0.0" iyy="0.0001" iyz="0.0" izz="0.0001"/>
+    </inertial>
+  </link>
+  <!-- Add a joint to attach the AprilTag to the drone -->
+  <joint name="apriltag_joint" type="fixed">
+    <parent link="main_body"/>
+    <child link="apriltag_link"/>
+    <origin xyz="0.1 0 -0.005"/>
+  </joint>
+  <!-- <xacro:extra_module name = "Apriltag_frame" parent = "main_body" visible = "1" > -->
+  <!--   <origin xyz=" 0.173 0.00 -0.008" rpy="0 ${pi} 0"/> -->
+  <!--   <inertial> -->
+  <!--     <mass value = "0.00001" /> -->
+  <!--     <origin xyz="0.1 0 -0.005" rpy="0 0 0"/> -->
+  <!--     <inertia -->
+  <!--         ixx="0.000001" ixy="0.0" ixz="0.0" -->
+  <!--         iyy="0.000001" iyz="0.0" -->
+  <!--         izz="0.000002"/>-\-> -->
+  <!--   </inertial> -->
+  <!-- </xacro:extra_module> -->
   <!-- propellers -->
   <xacro:propeller_module id = "1" x = "${-rotor_x}" y = "${-rotor_y}" z = "${rotor_z}" direction = "-1" />

Commit message: [Qilin][simulation] Show apriltag in gazebo

File: robots/mini_quadrotor/urdf/robot.urdf.xacro (robot description, xacro)
@@ -206,14 +206,11 @@
   <!--   </inertial> -->
   <!-- </xacro:extra_module> -->
-  <!-- New link for the AprilTag -->
+   <!-- New link for the AprilTag -->
   <link name="apriltag_link">
     <visual>
       <origin xyz="0 0 0" rpy="${-pi} 0 0"/>
       <geometry>
-        <box size="0.032 0.032 0.001"/>
-      </geometry>
-      <material name="apriltag_material">
-        <texture filename="package://aerial_robot_simulation/gazebo_model/models/Apriltag36_11_00000/materials/textures/tag36_11_00000.png"/>
-      </material>
+        <mesh filename="package://cooperation_landing/urdf/tag36_11_00000.dae" />
+      </geometry>
     </visual>
     <collision>
@@ -224,5 +221,5 @@
     </collision>
     <inertial>
-      <mass value="0.01"/>
+      <mass value="0.0001"/>
       <origin xyz="0 0 0"/>
       <inertia ixx="0.0001" ixy="0.0" ixz="0.0" iyy="0.0001" iyz="0.0" izz="0.0001"/>

Commit message: [Mini_quadrotor][urdf] Change LIDAR coordinate
In real world, I mount a protection shell for lidar. So I add 0.05 in z axis for LIDAR coordinate

File: robots/mini_quadrotor/urdf/robot.urdf.xacro (robot description, xacro)
@@ -163,5 +163,5 @@
   </xacro:extra_module>
   <xacro:extra_module name = "livox_link" parent = "main_body" visible = "0" >
-    <origin xyz="0 0 ${0.0425 + 0.047}" rpy="0 0 0"/>
+    <origin xyz="0 0 ${0.0425 + 0.047 + 0.005}" rpy="0 0 0"/>
     <inertial>
       <mass value = "0" />

Commit message: place the higher of lidar

File: robots/mini_quadrotor/urdf/robot.urdf.xacro (robot description, xacro)
@@ -153,5 +153,5 @@
   <!-- livox mid360 -->
   <xacro:extra_module name = "lidar_imu" parent = "main_body" visible = "0" > <!-- should be IMU frame -->
-    <origin xyz="${0.011} ${0.02329} ${0.0425 + 0.047 - 0.04412}" rpy="0 0 0"/> <!-- TODO: the true pos -->
+    <origin xyz="${0.011} ${0.02329} ${0.0425 + 0.047 - 0.04412 + 0.005}" rpy="0 0 0"/> <!-- TODO: the true pos -->
     <inertial>
       <mass value = "00" />

Commit message: [mini_quadrotor][simulation] Back to the begin state

File: robots/mini_quadrotor/urdf/robot.urdf.xacro (robot description, xacro)
@@ -206,24 +206,15 @@
   <!--   </inertial> -->
   <!-- </xacro:extra_module> -->
-   <!-- New link for the AprilTag -->
-  <link name="apriltag_link">
-    <visual>
-      <origin xyz="0 0 0" rpy="${-pi} 0 0"/>
-      <geometry>
-        <mesh filename="package://cooperation_landing/urdf/tag36_11_00000.dae" />
-      </geometry>
-    </visual>
-    <collision>
-      <origin xyz="0 0 0" rpy="0 0 0"/>
-      <geometry>
-        <box size="0.032 0.032 0.001"/>
-      </geometry>
-    </collision>
-    <inertial>
-      <mass value="0.0001"/>
-      <origin xyz="0 0 0"/>
-      <inertia ixx="0.0001" ixy="0.0" ixz="0.0" iyy="0.0001" iyz="0.0" izz="0.0001"/>
-    </inertial>
-  </link>
+  <!--  <!-\- New link for the AprilTag -\-> -->
+  <!-- <xacro:extra_module name = "apriltag_link" parent = "main_body" visible = "1" model_url = "package://cooperation_landing/urdf/tag36_11_00000.dae" > -->
+  <!--   <origin xyz="${0.1} 0 ${-0.005}" rpy="0 0 0"/> -->
+  <!--   <inertial> -->
+  <!--     <mass value = "0" /> -->
+  <!--     <origin xyz="0 0 0" rpy="${-pi} 0 0"/> -->
+  <!--     <inertia -->
+  <!--         ixx="0.0" ixy="0.0" ixz="0.0" -->
+  <!--         iyy="0.0" iyz="0.0" izz="0.0"/> -->
+  <!--   </inertial> -->
+  <!-- </xacro:extra_module> -->
   <!-- Add a joint to attach the AprilTag to the drone -->
   <joint name="apriltag_joint" type="fixed">
@@ -232,4 +223,23 @@
     <origin xyz="0.1 0 -0.005"/>
   </joint>
+  <link name="apriltag_link">
+    <visual>
+      <origin xyz="0 0 0" rpy="${-pi} 0 0"/>
+      <geometry>
+        <mesh filename="package://cooperation_landing/urdf/tag36_11_00000.dae" />
+      </geometry>
+    </visual>
+    <collision>
+      <origin xyz="0 0 0" rpy="0 0 0"/>
+      <geometry>
+        <box size="0.032 0.032 0.001"/>
+      </geometry>
+    </collision>
+    <inertial>
+      <mass value="0.0001"/>
+      <origin xyz="0 0 0"/>
+      <inertia ixx="0.0001" ixy="0.0" ixz="0.0" iyy="0.0001" iyz="0.0" izz="0.0001"/>
+    </inertial>
+  </link>
   <!-- <xacro:extra_module name = "Apriltag_frame" parent = "main_body" visible = "1" > -->
   <!--   <origin xyz=" 0.173 0.00 -0.008" rpy="0 ${pi} 0"/> -->

Commit message: [mini_quadrotor][urdf] Add apriltag

File: robots/mini_quadrotor/urdf/robot.urdf.xacro (robot description, xacro)
@@ -154,3 +154,28 @@
   <xacro:propeller_module id = "3" x = "${rotor_x}" y = "${rotor_y}" z = "${rotor_z}" direction = "-1" />
   <xacro:propeller_module id = "4" x = "${-rotor_x}" y = "${rotor_y}" z = "${rotor_z}"  direction = "1" />
+    <!-- Add a joint to attach the AprilTag to the drone -->
+  <joint name="apriltag_joint" type="fixed">
+    <parent link="main_body"/>
+    <child link="apriltag_link"/>
+    <origin xyz="0.1 0 -0.005"/>
+  </joint>
+  <link name="apriltag_link">
+    <visual>
+      <origin xyz="0 0 0" rpy="${-pi} 0 0"/>
+      <geometry>
+        <mesh filename="package://cooperation_landing/urdf/tag36_11_00000.dae" />
+      </geometry>
+    </visual>
+    <collision>
+      <origin xyz="0 0 0" rpy="0 0 0"/>
+      <geometry>
+        <box size="0.032 0.032 0.001"/>
+      </geometry>
+    </collision>
+    <inertial>
+      <mass value="0.0001"/>
+      <origin xyz="0 0 0"/>
+      <inertia ixx="0.0001" ixy="0.0" ixz="0.0" iyy="0.0001" iyz="0.0" izz="0.0001"/>
+    </inertial>
+  </link>
 </robot>

Commit message: Revert "[Modle][Control][Navigation] refactor the whole system from XYZ-Euler angles to true SO(3) (#671)"
This reverts commit 8db7e775a0be357e05124e9810bdb9c96704410f.

File: robots/mini_quadrotor/urdf/robot.urdf.xacro (robot description, xacro)
@@ -127,14 +127,4 @@
     </inertial>
   </xacro:extra_module>
-  <xacro:extra_module name = "magnet" parent = "main_body" visible = "0" >
-    <origin xyz="0 0 0" rpy="0 0 0"/>
-    <inertial>
-      <mass value = "00" />
-      <origin xyz="0 0 0" rpy="0 0 0"/>
-      <inertia
-          ixx="0.0" ixy="0.0" ixz="0.0"
-          iyy="0.0" iyz="0.0" izz="0.0"/>
-    </inertial>
-  </xacro:extra_module>
   <!-- livox mid360 -->
   <xacro:extra_module name = "lidar_imu" parent = "main_body" visible = "0" > <!-- should be IMU frame -->
