Commit message: [xuanwu][urdf] change the urdf file
Add the color and texture for xuanwu

File: robots/xuanwu/urdf/robot.urdf.xacro (robot description, xacro)
@@ -103,15 +103,15 @@
   <link name="main_body">
     <inertial>
-      <mass value = "0.747" />
-      <origin xyz="-0.00016 0.00010 0.03097" rpy="0 0 0"/> <!-- TODO: true cog pos -->
+      <mass value = "0.925" />
+      <origin xyz="0.00109 0.00008 0.01968" rpy="0 0 0"/> <!-- TODO: true cog pos -->
       <inertia
-          ixx="0.00527437131" ixy="0" ixz="0"
-          iyy="0.00537237336" iyz="0"
-          izz="0.00802880534"/>
+          ixx="0.00676315944" ixy="0" ixz="0"
+          iyy="0.00683176541" iyz="0"
+          izz="0.00882504031"/>
     </inertial>
     <visual>
       <origin rpy="0 0 0" xyz="0 0 0"/>
       <geometry>
-        <mesh filename="package://xuanwu/urdf/mesh/xuanwu_main_body_livox360.dae" />
+        <mesh filename="package://xuanwu/urdf/mesh/xuanwu_gripper_livox360.dae" />
       </geometry>
     </visual>
@@ -119,5 +119,5 @@
       <origin rpy="0 0 0" xyz="0 0 0"/>
       <geometry>
-        <box size="0.45227 0.45227 0.2248" />
+        <box size="0.45227 0.45227 0.2823" />
       </geometry>
     </collision>
@@ -125,5 +125,5 @@
   <!-- spinal -->
   <xacro:extra_module name = "fc" parent = "main_body" visible = "0" >
-    <origin xyz="-0.00016 0.00010 0.03097" rpy="0 0 0"/>
+    <origin xyz="0 0 0.0328" rpy="0 0 0"/>
     <inertial>
       <mass value = "00" />

Commit message: [xuanwu][LiDAR] edit the launch file and urdf

File: robots/xuanwu/urdf/robot.urdf.xacro (robot description, xacro)
@@ -134,4 +134,15 @@
     </inertial>
   </xacro:extra_module>
+  <!-- livox mid360 -->
+  <xacro:extra_module name = "lidar_imu" parent = "main_body" visible = "0" > <!-- should be IMU frame -->
+    <origin xyz="${0.011} ${0.02329} ${0.05879 + 0.047 - 0.04412}" rpy="0 0 0"/>
+    <inertial>
+      <mass value = "00" />
+      <origin xyz="0 0 0" rpy="0 0 0"/>
+      <inertia
+          ixx="0.0" ixy="0.0" ixz="0.0"
+          iyy="0.0" iyz="0.0" izz="0.0"/>
+    </inertial>
+  </xacro:extra_module>
   <!-- propellers -->
   <xacro:propeller_module id = "1" x = "${-rotor_x}" y = "${-rotor_y}" z = "${rotor_z}" direction = "1" />

Commit message: [xuanwu][urdf] Change the urdf file: Move the LiDAR`s IMU to spinal`s IMU. [xuanwu][urdf] Change the weight of main body: Add the LiDAR and gripper.

File: robots/xuanwu/urdf/robot.urdf.xacro (robot description, xacro)
@@ -103,5 +103,5 @@
   <link name="main_body">
     <inertial>
-      <mass value = "0.925" />
+      <mass value = "1.230" />
       <origin xyz="0.00109 0.00008 0.01968" rpy="0 0 0"/> <!-- TODO: true cog pos -->
       <inertia
@@ -136,5 +136,6 @@
   <!-- livox mid360 -->
   <xacro:extra_module name = "lidar_imu" parent = "main_body" visible = "0" > <!-- should be IMU frame -->
-    <origin xyz="${0.011} ${0.02329} ${0.05879 + 0.047 - 0.04412}" rpy="0 0 0"/>
+    <!-- <origin xyz="${0.011} ${0.02329} ${0.05879 + 0.047 - 0.04412}" rpy="0 0 0"/> -->
+    <origin xyz="0 0 0.0328" rpy="0 0 0"/>
     <inertial>
       <mass value = "00" />

Commit message: [xuanwu][urdf] change the urdf file, add the battery

File: robots/xuanwu/urdf/robot.urdf.xacro (robot description, xacro)
@@ -103,10 +103,10 @@
   <link name="main_body">
     <inertial>
-      <mass value = "1.230" />
-      <origin xyz="0.00109 0.00008 0.01968" rpy="0 0 0"/> <!-- TODO: true cog pos -->
+      <mass value = "1.6426" />
+      <origin xyz="0.01319 -0.000007 -0.00426" rpy="0 0 0"/> <!-- TODO: true cog pos -->
       <inertia
-          ixx="0.00676315944" ixy="0" ixz="0"
-          iyy="0.00683176541" iyz="0"
-          izz="0.00882504031"/>
+          ixx="0.01075808343" ixy="0" ixz="0"
+          iyy="0.01067287487" iyz="0"
+          izz="0.01227783623"/>
     </inertial>
     <visual>
@@ -119,5 +119,5 @@
       <origin rpy="0 0 0" xyz="0 0 0"/>
       <geometry>
-        <box size="0.45227 0.45227 0.2823" />
+        <box size="0.45227 0.45227 0.2295" />
       </geometry>
     </collision>

Commit message: [xuanwu][urdf] change the mesh file

File: robots/xuanwu/urdf/robot.urdf.xacro (robot description, xacro)
@@ -113,5 +113,5 @@
       <origin rpy="0 0 0" xyz="0 0 0"/>
       <geometry>
-        <mesh filename="package://xuanwu/urdf/mesh/xuanwu_gripper_livox360.dae" />
+        <mesh filename="package://xuanwu/urdf/mesh/drone_gripper_battery_LiDAR.dae" />
       </geometry>
     </visual>

Commit message: [urdf] Change the model to 1300 mAh batteries

File: robots/xuanwu/urdf/robot.urdf.xacro (robot description, xacro)
@@ -103,15 +103,15 @@
   <link name="main_body">
     <inertial>
-      <mass value = "1.6426" />
-      <origin xyz="0.01319 -0.000007 -0.00426" rpy="0 0 0"/> <!-- TODO: true cog pos -->
+      <mass value = "1.666" />
+      <origin xyz="0.00093 -0.00007 -0.00477" rpy="0 0 0"/> <!-- TODO: true cog pos -->
       <inertia
-          ixx="0.01075808343" ixy="0" ixz="0"
-          iyy="0.01067287487" iyz="0"
-          izz="0.01227783623"/>
+          ixx="0.01079536794" ixy="0" ixz="0"
+          iyy="0.01024013115" iyz="0"
+          izz="0.01187755262"/>
     </inertial>
     <visual>
       <origin rpy="0 0 0" xyz="0 0 0"/>
       <geometry>
-        <mesh filename="package://xuanwu/urdf/mesh/drone_gripper_battery_LiDAR.dae" />
+        <mesh filename="package://xuanwu/urdf/mesh/drone_gripper_battery_LiDAR_1300.dae" />
       </geometry>
     </visual>

Commit message: [xuanwu][urdf] change the urdf with camera

File: robots/xuanwu/urdf/robot.urdf.xacro (robot description, xacro)
@@ -104,9 +104,9 @@
     <inertial>
       <mass value = "1.666" />
-      <origin xyz="0.00093 -0.00007 -0.00477" rpy="0 0 0"/> <!-- TODO: true cog pos -->
+      <origin xyz="0.00132 0.00007 -0.00738" rpy="0 0 0"/>
       <inertia
-          ixx="0.01079536794" ixy="0" ixz="0"
-          iyy="0.01024013115" iyz="0"
-          izz="0.01187755262"/>
+          ixx="0.01171975383" ixy="0" ixz="0"
+          iyy="0.01269245515" iyz="0"
+          izz="0.01115712375"/>
     </inertial>
     <visual>
@@ -119,5 +119,5 @@
       <origin rpy="0 0 0" xyz="0 0 0"/>
       <geometry>
-        <box size="0.45227 0.45227 0.2295" />
+        <box size="0.45227 0.45227 0.2853" />
       </geometry>
     </collision>

Commit message: [xuanwu][urdf] Update the drone model and changed mocap sensor unhealth level.

File: robots/xuanwu/urdf/robot.urdf.xacro (robot description, xacro)
@@ -6,7 +6,7 @@
   <thrust_link name="thrust" />
   <!-- kinematics [m] -->!!!!!!!!!!!!!
-  <xacro:property name="rotor_x" value="0.11314" />
-  <xacro:property name="rotor_y" value="0.11314" />
-  <xacro:property name="rotor_z" value="0.0415" />
+  <xacro:property name="rotor_x" value="0.12728" />
+  <xacro:property name="rotor_y" value="0.12731" />
+  <xacro:property name="rotor_z" value="0.036" />
   <!-- dynamics -->
   <m_f_rate value="-0.011" /> <!-- drag torque rate -->
@@ -103,10 +103,10 @@
   <link name="main_body">
     <inertial>
-      <mass value = "1.666" />
-      <origin xyz="0.00132 0.00007 -0.00738" rpy="0 0 0"/>
+      <mass value = "1.767" />
+      <origin xyz="0.0013 0.00004 -0.00754" rpy="0 0 0"/>
       <inertia
-          ixx="0.01171975383" ixy="0" ixz="0"
-          iyy="0.01269245515" iyz="0"
-          izz="0.01115712375"/>
+          ixx="0.01319022271" ixy="0" ixz="0"
+          iyy="0.01262070107" iyz="0"
+          izz="0.01546757494"/>
     </inertial>
     <visual>
@@ -119,5 +119,5 @@
       <origin rpy="0 0 0" xyz="0 0 0"/>
       <geometry>
-        <box size="0.45227 0.45227 0.2853" />
+        <box size="0.48064 0.48064 0.2853" />
       </geometry>
     </collision>

Commit message: Implements the ESKF and allows dynamic param tunning

File: robots/xuanwu/urdf/robot.urdf.xacro (robot description, xacro)
@@ -148,5 +148,5 @@
   <!-- downward camera -->
   <xacro:extra_module name = "aerial_robot_camera_frame" parent = "main_body" visible = "0" >
-    <origin xyz="-0.003 0 -0.1042" rpy="0 0 0"/>
+	  <origin xyz="-0.003 0 -0.1042" rpy="0 ${pi} ${-pi/2}"/>
     <inertial>
       <mass value = "0.00001" />
@@ -158,5 +158,5 @@
   </xacro:extra_module>
   <xacro:extra_module name = "aerial_robot_camera_optical_frame" parent = "aerial_robot_camera_frame" visible = "0" >
-    <origin xyz="0 0 0" rpy="0 ${pi/2} 0"/>
+	  <origin xyz="0 0 0" rpy="0 ${-pi/2} ${pi/2}"/>
     <inertial>
       <mass value = "0.00001" />

Commit message: Adjusts landing criteria and updates camera position

File: robots/xuanwu/urdf/robot.urdf.xacro (robot description, xacro)
@@ -148,5 +148,5 @@
   <!-- downward camera -->
   <xacro:extra_module name = "aerial_robot_camera_frame" parent = "main_body" visible = "0" >
-	  <origin xyz="-0.003 0 -0.1042" rpy="0 ${pi} ${-pi/2}"/>
+	  <origin xyz="-0.003 0 -0.159" rpy="0 ${pi} ${-pi/2}"/>
     <inertial>
       <mass value = "0.00001" />

Commit message: [code] storage

File: robots/xuanwu/urdf/robot.urdf.xacro (robot description, xacro)
@@ -148,5 +148,5 @@
   <!-- downward camera -->
   <xacro:extra_module name = "aerial_robot_camera_frame" parent = "main_body" visible = "0" >
-	  <origin xyz="-0.003 0 -0.1042" rpy="0 ${pi} ${-pi/2}"/>
+	  <origin xyz="-0.003 0 -0.16" rpy="0 ${pi} ${-pi/2}"/>
     <inertial>
       <mass value = "0.00001" />

Commit message: Match the camera_frame between launch file and urdf.

File: robots/xuanwu/urdf/robot.urdf.xacro (robot description, xacro)
@@ -111,5 +111,5 @@
     </inertial>
     <visual>
-      <origin rpy="0 0 0" xyz="0 0 0"/>
+      <origin rpy="0 0 ${pi}" xyz="0 0 0"/>
       <geometry>
         <mesh filename="package://xuanwu/urdf/mesh/drone_gripper_battery_LiDAR_1300_gripper_180mm.dae" />
@@ -146,4 +146,25 @@
     </inertial>
   </xacro:extra_module>
+  <!-- forward camera -->
+  <xacro:extra_module name = "aerial_robot_camera_frame" parent = "main_body" visible = "0" >
+	  <origin xyz="0.05798 0 -0.047" rpy="0 0 0"/>
+    <inertial>
+      <mass value = "0.00001" />
+      <origin xyz="0 0 0" rpy="0 0 0"/>
+      <inertia
+          ixx="0.0" ixy="0.0" ixz="0.0"
+          iyy="0.0" iyz="0.0" izz="0.0"/>
+    </inertial>
+  </xacro:extra_module>
+  <xacro:extra_module name = "aerial_robot_camera_optical_frame" parent = "aerial_robot_camera_frame" visible = "0" >
+	  <origin xyz="0 0 0" rpy="${-pi/2} 0 ${-pi/2}"/>
+    <inertial>
+      <mass value = "0.00001" />
+      <origin xyz="0 0 0" rpy="0 0 0"/>
+      <inertia
+          ixx="0.0" ixy="0.0" ixz="0.0"
+          iyy="0.0" iyz="0.0" izz="0.0"/>
+    </inertial>
+  </xacro:extra_module>
   <!-- propellers -->
   <xacro:propeller_module id = "1" x = "${-rotor_x}" y = "${-rotor_y}" z = "${rotor_z}" direction = "1" />

Commit message: [xuanwu][urdf] Change the cog position.

File: robots/xuanwu/urdf/robot.urdf.xacro (robot description, xacro)
@@ -104,5 +104,5 @@
     <inertial>
       <mass value = "1.900" />
-      <origin xyz="0.00147 -0.00007 -0.01451" rpy="0 0 0"/>
+      <origin xyz="-0.013 -0.00507 -0.01451" rpy="0 0 0"/>
       <inertia
           ixx="0.01400956434" ixy="0" ixz="0"

Commit message: [xuanwu][urdf] Change the model forward direction.

File: robots/xuanwu/urdf/robot.urdf.xacro (robot description, xacro)
@@ -111,5 +111,5 @@
     </inertial>
     <visual>
-      <origin rpy="0 0 ${pi}" xyz="0 0 0"/>
+      <origin rpy="0 0 0" xyz="0 0 0"/>
       <geometry>
         <mesh filename="package://xuanwu/urdf/mesh/drone_gripper_battery_LiDAR_1300_gripper_180mm.dae" />
