Commit message: [xuanwu][config] update the coordinate transform matrix. [urdf] Update the cog with LiHv batt

File: robots/xuanwu/urdf/robot.urdf.xacro (robot description, xacro)
@@ -104,5 +104,5 @@
     <inertial>
       <mass value = "1.900" />
-      <origin xyz="-0.013 -0.00507 -0.01451" rpy="0 0 0"/>
+      <origin xyz="-0.013 -0.01007 -0.01451" rpy="0 0 0"/>
       <inertia
           ixx="0.01400956434" ixy="0" ixz="0"
